File: AS_Upcvt.sch (KiCad schematic (older format))
At the start: 24 parts, among them P1 BNC, P2 BNC, P3 BNC, T1 TUF-2LHSM, T2 FE-735M

Commit message: changed Readme
Other:
- note added: "OL In \n779 MHz"
Changed lines of the file:
@@
 LIBS:switches
 LIBS:transistors
-LIBS:tuf-2lhsm
 LIBS:AS_Upcvt-cache
 EELAYER 25 0
@@
 Wire Wire Line
 	4900 1900 4900 1950
+Text Notes 5200 2050 1    60   ~ 0
+OL In \n779 MHz
 $EndSCHEMATC

Commit message: documentation added
Parts:
- T2: value FE-735M -> 302HXPK-1341D1
Other:
- note added: "All caps C0G\nAll inductance Wurth wire wound\nall UHF branches with 0603 components"
- note added: "LPF 700 MHz\nOut 779 – 928 MHz\nTO Texas S.A."
- note added: "OL Input\n779 MHz"
- note added: "Signal in \n1-149 MHz"
- note added: "Upconverter for the\nTexas Instrument sub GHz spectrum analyzer\nMSP-SA430-SUB1GHZ"
- note added: "triple helical filter\ndigikey TK3409-ND"
- note removed: "LPF 700 MHz\nOut 779 – 928 MHz"
- note removed: "OL In \n779 MHz"
- note removed: "in 1-149 MHz"
Changed lines of the file:
@@
 LIBS:switches
 LIBS:transistors
+LIBS:tuf-2lhsm
 LIBS:AS_Upcvt-cache
 EELAYER 25 0
@@
 Wire Wire Line
 	3250 3350 3250 3400
-Text Notes 500  1750 0    60   ~ 0
-in 1-149 MHz
+Text Notes 1150 1400 0    60   ~ 0
+Signal in \n1-149 MHz
 Text Notes 3050 3950 0    60   ~ 0
-LPF 700 MHz\nOut 779 – 928 MHz
+LPF 700 MHz\nOut 779 – 928 MHz\nTO Texas S.A.
 $Comp
 L GND #PWR7
@@
 P 4100 1500
 F 0 "T2" H 4100 1750 50  0000 C CNN
-F 1 "FE-735M" H 4100 1200 50  0000 C CNN
+F 1 "302HXPK-1341D1" H 4100 1200 50  0000 C CNN
 F 2 "" H 4100 1500 50  0001 C CNN
 F 3 "" H 4100 1500 50  0001 C CNN
@@
 Wire Wire Line
 	4900 1900 4900 1950
-Text Notes 5200 2050 1    60   ~ 0
-OL In \n779 MHz
+Text Notes 5500 1850 2    60   ~ 0
+OL Input\n779 MHz
+Text Notes 4800 1350 0    60   ~ 0
+triple helical filter\ndigikey TK3409-ND
+Text Notes 5600 3750 0    60   ~ 0
+All caps C0G\nAll inductance Wurth wire wound\nall UHF branches with 0603 components
+Text Notes 7150 6850 0    60   ~ 0
+Upconverter for the\nTexas Instrument  sub GHz spectrum analyzer\nMSP-SA430-SUB1GHZ
 $EndSCHEMATC
